File: retro-ingenerieDS3231.kicad_sch (KiCad schematic)
At the start: 14 parts

Commit message: Add files via upload
Parts:
- removed RN1, RN2: R_Network04_US, Resistor_THT:R_Array_SIP5, symbol Device:R_Network04_US
- removed U2: ~, symbol New_Library:selecteur_d'adressse_EEPROM
- removed U3: ~, symbol New_Library:DS3231
- added RN1: 4*4,7K, Resistor_SMD:R_Array_Convex_4x0603, symbol Device:R_Pack04
- added RN3: 4*4,7k, Resistor_SMD:R_Array_Convex_4x0603, symbol Device:R_Pack04
- added U2: DS3231, Library_kiady:SOIC -16, symbol New_Library:DS3231
- added U3: ~, Library_kiady:EEPROM_Adress_Selector_3xSJ, symbol New_Library:selecteur_d'adressse_EEPROM
- BT1: value Battery -> CR2032 OU LIR2032; footprint (none) -> Battery:BatteryHolder_Keystone_1060_1x2032
- C1, C2: footprint (none) -> Capacitor_SMD:C_0805_2012Metric
- CN1: footprint (none) -> Connector_PinHeader_2.54mm:PinHeader_1x06_P2.54mm_Vertical
- CN2: footprint (none) -> Connector_PinHeader_2.54mm:PinHeader_1x04_P2.54mm_Vertical
- D1: footprint (none) -> LED_SMD:LED_0805_2012Metric
- D2: footprint Diode_THT:D_DO-35_SOD27_P7.62mm_Horizontal -> Diode_SMD:D_SOD-123
- R1: renamed from R2; footprint (none) -> Resistor_SMD:R_0805_2012Metric
- R2: renamed from R1; value R -> 1k; footprint (none) -> Resistor_SMD:R_0805_2012Metric
- U1: value ~ -> AT24C32; footprint (none) -> Library_kiady:SOIC -8
Connections:
- net 32K: now also CN1.1, RN1.1 (R1.1), U2.1 (32kHz); no longer CN1. (6)
- net GND: now also CN1.6, CN2.4, U2.13 (GND), U3.4, U3.5, U3.6; no longer CN1. (6)
- net SCL: now also CN1.3, CN2.1, RN1.3 (R3.1), U2.16 (SCL); no longer CN1. (6)
- net SDA: now also CN1.4, CN2.2, RN1.4 (R4.1), U2.15 (SDA); no longer CN1. (6)
- net SQW: now also CN1.2, RN1.2 (R2.1), U2.3 (INTSQW); no longer CN1. (6)
- net VCC: now also CN1.5, CN2.3, RN1.5 (R4.2), RN1.6 (R3.2), RN1.7 (R2.2), RN1.8 (R1.2), RN3.5 (R4.2), RN3.6 (R3.2), RN3.7 (R2.2), RN3.8 (R1.2); no longer BT1.1 (+), CN1. (6), D2.1 (K)
- net A0: now reaches U1.1 (A0)
- net A0: now also RN3.2 (R2.1), U3.1
- net A1: now reaches U1.2 (A1)
- net A1: now also RN3.3 (R3.1), U3.2
- net A2: now reaches U1.3 (A2)
- net A2: now also RN3.4 (R4.1), U3.3
- new net: BT1.1 (+), D2.1 (K), U2.2 (VCC)
Other:
- note added: "08/07/2026"
- note added: "Module DS3231"
